Commit message: Add bottom camera

File: bubbles_description/urdf/bubbles_sensors.xacro (robot description, xacro)
@@ -29,4 +29,20 @@
       <origin xyz="0.2 0 0.0" rpy="0 0 0"/>
   </xacro:regular_camera_plugin_macro>
+  <!-- Bottom Camera -->
+ <xacro:regular_camera_plugin_macro
+      namespace="${namespace}"
+      suffix="_bottom"
+      parent_link="${namespace}/base_link"
+      topic="camera"
+      mass="0.0001"
+      update_rate="30"
+      hfov="1.8125"
+      width="1920"
+      height="1080"
+      stddev="0.02"
+      scale="0.5">
+      <inertia ixx="0.00001" ixy="0.0" ixz="0.0" iyy="0.00001" iyz="0.0" izz="0.00001" />
+      <origin xyz="0.0 0.0 -0.07" rpy="0 1.57 0"/>
+  </xacro:regular_camera_plugin_macro>
   <!-- IMU  -->
   <xacro:default_imu_macro
